File: box.brd (EAGLE design)
At the start: 100 x 80 mm, 38 parts, among them U1 SN74HC266N, U2 SN74HC266N, U3 SN74HC266N

Commit message: PCB ok
Parts:
- added D1: (no value), diode:DO41-7.6
- added E$1, E$3, E$5: (no value), fabBox:LOGO_200
- added E$2, E$4, E$6, U$1, U$2, U$3: (no value), fabBox:LOGO_200_TEXT
- added JP1: (no value), SparkFun-Connectors:JST-2-PTH
- added PAD1, PAD13, PAD14, PAD2, PAD7, PAD8: +, wirepad:2,15/1,0
- added PAD10, PAD15, PAD16, PAD3, PAD4, PAD9: ERROR, wirepad:2,15/1,0
- added PAD11, PAD12, PAD17, PAD18, PAD5, PAD6: -, wirepad:2,15/1,0
- C1, C2, C3: value (none) -> 100n
- moved T1 162.0 mm to (79.6, 38.0), turned to 90 degrees
- moved U3 153.9 mm to (85.7, 56.7)
- moved R23 151.9 mm to (79.4, 51.6), turned to 270 degrees
- moved R22 144.3 mm to (76.8, 51.6), turned to 270 degrees
- moved R19 136.7 mm to (84.5, 51.6), turned to 270 degrees
- moved R21 134.2 mm to (71.8, 51.6), turned to 270 degrees
- moved R20 126.5 mm to (69.2, 51.6), turned to 270 degrees
- moved SW6 126.5 mm to (70.5, 65.6), turned to 90 degrees
- moved R11 125.3 mm to (54.0, 51.6), turned to 270 degrees
- moved R18 121.5 mm to (74.3, 51.6), turned to 270 degrees
- moved SW5 110.2 mm to (70.5, 65.6), flipped to the bottom, turned to 90 degrees
- moved R10 110.1 mm to (43.8, 51.6), turned to 270 degrees
- moved R25 110.0 mm to (85.1, 38.1)
- moved U2 108.3 mm to (55.2, 56.7)
- moved R17 108.0 mm to (66.0, 55.4), turned to 270 degrees
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Connections:
- new net N$26: R24.1, SW6.8, U3.13
- net /ERROR: now also PAD10.1, PAD15.1, PAD16.1, PAD3.1, PAD4.1, PAD9.1, T1.3
- net GND: now also PAD11.1, PAD12.1, PAD17.1, PAD18.1, PAD5.1, PAD6.1, T1.4
- net N$1: now also SW1.1; no longer SW1.8
- net N$10: now also R9.1, SW3.1, U2.1; no longer R10.1, SW3.4, U2.5
- net N$11: now also R10.1, U2.5; no longer R11.1, U2.8
- net N$12: now also R11.1, SW3.4, U2.8; no longer R12.1, SW3.1, U2.12
- net N$13: now also R12.1, SW3.8, U2.12; no longer R13.1, SW4.8, U2.2
- net N$14: now also R13.1, SW4.1, U2.2; no longer R14.1, SW4.4, U2.6
- net N$15: now also R14.1, U2.6; no longer R15.1, U2.9
- net N$16: now also R15.1, SW4.4, U2.9; no longer R16.1, SW4.1, U2.13
- net N$17: now also R16.1, SW4.8, U2.13; no longer R17.1, SW5.8, U3.1
- net N$18: now also R17.1, SW5.1, U3.1; no longer R18.1, SW5.4, U3.5
- net N$19: now also R18.1, U3.5; no longer R19.1, U3.8
- net N$2: now also SW1.2; no longer SW1.4
- net N$20: now also R19.1, SW5.4, U3.8; no longer R20.1, SW5.1, U3.12
- net N$21: now also R20.1, SW5.8, U3.12; no longer R21.1, SW6.8, U3.2
- net N$22: now also R21.1, SW6.1, U3.2; no longer R22.1, SW6.4, U3.6
- net N$23: now also R22.1, U3.6; no longer R23.1, U3.9
- net N$24: now also R23.1, SW6.4, U3.9; no longer R24.1, SW6.1, U3.13
- net N$3: now also SW1.4; no longer SW1.2
- net N$4: now also SW1.8; no longer SW1.1
- net N$5: now also D1.A, JP1.1, T1.1, T1.2, T1.5, T1.6; no longer R9.1, SW3.8, U2.1
- net N$6: now also SW2.1; no longer SW2.8
- net N$7: now also SW2.2; no longer SW2.4
- net N$8: now also SW2.4; no longer SW2.2
- net N$9: now also SW2.8; no longer SW2.1
- net VCC: now also D1.C, JP1.2, PAD1.1, PAD13.1, PAD14.1, PAD2.1, PAD7.1, PAD8.1
Routing:
- net /ERROR: track 0.00 -> 142.2 mm, vias 0 -> 9
- net VCC: track 0.00 -> 115.6 mm
- net GND: track 0.00 -> 68.2 mm, vias 0 -> 5
- net N$8: track 0.00 -> 42.1 mm, vias 0 -> 3
- net N$24: track 0.00 -> 42.1 mm, vias 0 -> 3
- net N$16: track 0.00 -> 42.1 mm, vias 0 -> 3
- net N$22: track 0.00 -> 39.5 mm, vias 0 -> 4
- net N$14: track 0.00 -> 38.4 mm, vias 0 -> 4
- net N$6: track 0.00 -> 38.4 mm, vias 0 -> 4
- net N$18: track 0.00 -> 38.0 mm, vias 0 -> 4
- net N$10: track 0.00 -> 38.0 mm, vias 0 -> 4
- net N$1: track 0.00 -> 38.0 mm, vias 0 -> 4
- net N$26: track 0.00 -> 37.4 mm, vias 0 -> 3
- net N$9: track 0.00 -> 36.3 mm, vias 0 -> 3
- net N$17: track 0.00 -> 36.3 mm, vias 0 -> 3
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- added copper zone on layer 16, net GND
- added copper zone on layer 1, net VCC
Other:
- board size 100 x 80 mm -> 91 x 45 mm
- board text added: "100n"
- board text added: "8x10k"
- board text added: "FabBox"
- board text added: "Partial vertical slots"
