File: box.sch (EAGLE design)
At the start: 38 parts, among them U1 SN74HC266N, U2 SN74HC266N, U3 SN74HC266N

Commit message: PCB ok
Parts:
- added D1: (no value), diode:DIODE-DO41-7.6
- added JP1: (no value), SparkFun-Connectors:M02JST-PTH-2
- added PAD1, PAD13, PAD14, PAD2, PAD7, PAD8: +, wirepad:2,15/1,0
- added PAD10, PAD15, PAD16, PAD3, PAD4, PAD9: ERROR, wirepad:2,15/1,0
- added PAD11, PAD12, PAD17, PAD18, PAD5, PAD6: -, wirepad:2,15/1,0
- C1, C2, C3: value (none) -> 100n
Connections:
- new net N$26: R24.1, SW6.8, U3.4B
- net /ERROR: now also PAD10.P, PAD15.P, PAD16.P, PAD3.P, PAD4.P, PAD9.P, T1.G
- net GND: now also PAD11.P, PAD12.P, PAD17.P, PAD18.P, PAD5.P, PAD6.P, T1.S
- net N$1: now also SW1.1; no longer SW1.8
- net N$10: now also R9.1, SW3.1, U2.1A; no longer R10.1, SW3.4, U2.2A
- net N$11: now also R10.1, U2.2A; no longer R11.1, U2.3A
- net N$12: now also R11.1, SW3.4, U2.3A; no longer R12.1, SW3.1, U2.4A
- net N$13: now also R12.1, SW3.8, U2.4A; no longer R13.1, SW4.8, U2.1B
- net N$14: now also R13.1, SW4.1, U2.1B; no longer R14.1, SW4.4, U2.2B
- net N$15: now also R14.1, U2.2B; no longer R15.1, U2.3B
- net N$16: now also R15.1, SW4.4, U2.3B; no longer R16.1, SW4.1, U2.4B
- net N$17: now also R16.1, SW4.8, U2.4B; no longer R17.1, SW5.8, U3.1A
- net N$18: now also R17.1, SW5.1, U3.1A; no longer R18.1, SW5.4, U3.2A
- net N$19: now also R18.1, U3.2A; no longer R19.1, U3.3A
- net N$2: now also SW1.2; no longer SW1.4
- net N$20: now also R19.1, SW5.4, U3.3A; no longer R20.1, SW5.1, U3.4A
- net N$21: now also R20.1, SW5.8, U3.4A; no longer R21.1, SW6.8, U3.1B
- net N$22: now also R21.1, SW6.1, U3.1B; no longer R22.1, SW6.4, U3.2B
- net N$23: now also R22.1, U3.2B; no longer R23.1, U3.3B
- net N$24: now also R23.1, SW6.4, U3.3B; no longer R24.1, SW6.1, U3.4B
- net N$3: now also SW1.4; no longer SW1.2
- net N$4: now also SW1.8; no longer SW1.1
- net N$5: now also D1.A, JP1.1, T1.D; no longer R9.1, SW3.8, U2.1A
- net N$6: now also SW2.1; no longer SW2.8
- net N$7: now also SW2.2; no longer SW2.4
- net N$8: now also SW2.4; no longer SW2.2
- net N$9: now also SW2.8; no longer SW2.1
- net VCC: now also D1.C, JP1.2, PAD1.P, PAD13.P, PAD14.P, PAD2.P, PAD7.P, PAD8.P
Other:
- moved on the sheet: C2, C3, R10, R11, R12, R13, R14, R15, R16, R17, R18, R19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
